File: hardware/sound-generator-board/sgb.sch (KiCad schematic (older format))
At the start: 35 parts, among them P1 CONN_5, P2 CONN_5, P3 CONN_2X2, P4 CONN_6, P5 CONN_4, P6 CONN_4, P7 CONN_5, P8 CONN_5, Q1 NPN, U1 AY-3-8912, U2 74LS139, U3 74HC04, U4 AY-3-8912, U5 AY-3-8912, U6 AY-3-8912

Commit message: Initial sound generator board done
Parts:
- removed P3: CONN_2X2, symbol CONN_2X2
- added C4: 100µF, symbol CP1
- added C5: C, symbol C
- added D1, D2: DIODE, symbol DIODE
- added K1: CONN_3, symbol CONN_3
- added P10, P11, P12, P13, P14, P9: CONN_4, symbol CONN_4
- added Q2: BC182, TO92, symbol BC547
- added R16, R19: 10kΩ, symbol R
- added R17: 680Ω, symbol R
- added R18: 8.2kΩ, symbol R
Connections:
- net labels added: IO0, IO1, IO10, IO11, IO12, IO13, IO14, IO15, IO16, IO17, IO2, IO20, IO21, IO22, IO23, IO24, IO25, IO26, IO27, IO3, IO30, IO31, IO32, IO33, IO34, IO35, IO36, IO37, IO4, IO5, IO6, IO7, MIX_LINE_IN, MIX_OUT
- wire segments 247 -> 336
Other:
- moved on the sheet: P5, P6

Commit message: Forgot to add decoupling to 3 of the sound generators
Parts:
- added C6, C7, C8: C, symbol C
Connections:
- net GND: now also C6.2, C7.2, C8.2
- net VCC: now also C6.1, C7.1, C8.1
Changed lines of the file:
@@
-EESchema Schematic File Version 2  date Sat 03 Aug 2013 01:23:42 PM CEST
+EESchema Schematic File Version 2  date Sat 03 Aug 2013 01:38:29 PM CEST
 LIBS:power
 LIBS:device
@@
 Comment4 ""
 $EndDescr
+Connection ~ 5700 1750
+Wire Wire Line
+	5950 1750 5450 1750
+Wire Wire Line
+	5700 1750 5700 1950
 Wire Wire Line
 	3650 5250 3650 5350
@@
 Wire Wire Line
 	3850 5100 3850 5250
+Wire Wire Line
+	5700 1350 5700 1100
+Wire Wire Line
+	5950 1350 5450 1350
+Connection ~ 5700 1350
+$Comp
+L VCC #PWR9
+U 1 1 51FCEAE9
+P 5700 1100
+F 0 "#PWR9" H 5700 1200 30  0001 C CNN
+F 1 "VCC" H 5700 1200 30  0000 C CNN
+	1    5700 1100
+	1    0    0    -1
+$EndComp
+$Comp
+L GND #PWR10
+U 1 1 51FCEAE1
+P 5700 1950
+F 0 "#PWR10" H 5700 1950 30  0001 C CNN
+F 1 "GND" H 5700 1880 30  0001 C CNN
+	1    5700 1950
+	1    0    0    -1
+$EndComp
+$Comp
+L C C8
+U 1 1 51FCEAD4
+P 5950 1550
+F 0 "C8" H 6000 1650 50  0000 L CNN
+F 1 "C" H 6000 1450 50  0000 L CNN
+	1    5950 1550
+	1    0    0    -1
+$EndComp
+$Comp
+L C C7
+U 1 1 51FCEAD0
+P 5700 1550
+F 0 "C7" H 5750 1650 50  0000 L CNN
+F 1 "C" H 5750 1450 50  0000 L CNN
+	1    5700 1550
+	1    0    0    -1
+$EndComp
+$Comp
+L C C6
+U 1 1 51FCEACE
+P 5450 1550
+F 0 "C6" H 5500 1650 50  0000 L CNN
+F 1 "C" H 5500 1450 50  0000 L CNN
+	1    5450 1550
+	1    0    0    -1
+$EndComp
 $Comp
 L CONN_3 K1
@@
 $EndComp
 $Comp
-L VCC #PWR01
+L VCC #PWR5
 U 1 1 51FCD7A5
 P 3350 1200
-F 0 "#PWR01" H 3350 1300 30  0001 C CNN
+F 0 "#PWR5" H 3350 1300 30  0001 C CNN
 F 1 "VCC" H 3350 1300 30  0000 C CNN
 	1    3350 1200
@@
 $EndComp
 $Comp
-L GND #PWR02
+L GND #PWR6
 U 1 1 51FCD79B
 P 3950 2500
-F 0 "#PWR02" H 3950 2500 30  0001 C CNN
+F 0 "#PWR6" H 3950 2500 30  0001 C CNN
 F 1 "GND" H 3950 2430 30  0001 C CNN
 	1    3950 2500
@@
 DA0
 $Comp
-L GND #PWR03
+L GND #PWR13
 U 1 1 51FBF4B9
 P 9900 2450
-F 0 "#PWR03" H 9900 2450 30  0001 C CNN
+F 0 "#PWR13" H 9900 2450 30  0001 C CNN
 F 1 "GND" H 9900 2380 30  0001 C CNN
 	1    9900 2450
@@
 $EndComp
 $Comp
-L VCC #PWR04
+L VCC #PWR14
 U 1 1 51FBF4B1
 P 9900 2550
-F 0 "#PWR04" H 9900 2650 30  0001 C CNN
+F 0 "#PWR14" H 9900 2650 30  0001 C CNN
 F 1 "VCC" H 9900 2650 30  0000 C CNN
 	1    9900 2550
@@
 $EndComp
 $Comp
-L VCC #PWR05
+L VCC #PWR12
 U 1 1 51FBF44C
 P 9700 4700
-F 0 "#PWR05" H 9700 4800 30  0001 C CNN
+F 0 "#PWR12" H 9700 4800 30  0001 C CNN
 F 1 "VCC" H 9700 4800 30  0000 C CNN
 	1    9700 4700
@@
 $EndComp
 $Comp
-L GND #PWR06
+L GND #PWR11
 U 1 1 51FBF43F
 P 9600 4700
-F 0 "#PWR06" H 9600 4700 30  0001 C CNN
+F 0 "#PWR11" H 9600 4700 30  0001 C CNN
 F 1 "GND" H 9600 4630 30  0001 C CNN
 	1    9600 4700
@@
 $EndComp
 $Comp
-L GND #PWR07
+L GND #PWR8
 U 1 1 51967238
 P 5400 4650
-F 0 "#PWR07" H 5400 4650 30  0001 C CNN
+F 0 "#PWR8" H 5400 4650 30  0001 C CNN
 F 1 "GND" H 5400 4580 30  0001 C CNN
 	1    5400 4650
@@
 $EndComp
 $Comp
-L GND #PWR08
+L GND #PWR4
 U 1 1 51967005
 P 3200 4200
-F 0 "#PWR08" H 3200 4200 30  0001 C CNN
+F 0 "#PWR4" H 3200 4200 30  0001 C CNN
 F 1 "GND" H 3200 4130 30  0001 C CNN
 	1    3200 4200
@@
 $EndComp
 $Comp
-L VCC #PWR09
+L VCC #PWR3
 U 1 1 51967001
 P 3150 4100
-F 0 "#PWR09" H 3150 4200 30  0001 C CNN
+F 0 "#PWR3" H 3150 4200 30  0001 C CNN
 F 1 "VCC" H 3150 4200 30  0000 C CNN
 	1    3150 4100
@@
 $EndComp
 $Comp
-L GND #PWR010
+L GND #PWR2
 U 1 1 51966E52
 P 2200 7700
-F 0 "#PWR010" H 2200 7700 30  0001 C CNN
+F 0 "#PWR2" H 2200 7700 30  0001 C CNN
 F 1 "GND" H 2200 7630 30  0001 C CNN
 	1    2200 7700
@@
 $EndComp
 $Comp
-L VCC #PWR011
+L VCC #PWR1
 U 1 1 51966E3F
 P 900 7650
-F 0 "#PWR011" H 900 7750 30  0001 C CNN
+F 0 "#PWR1" H 900 7750 30  0001 C CNN
 F 1 "VCC" H 900 7750 30  0000 C CNN
 	1    900  7650
@@
 $EndComp
 $Comp
-L VCC #PWR012
+L VCC #PWR7
 U 1 1 517CEB07
 P 4850 4350
-F 0 "#PWR012" H 4850 4450 30  0001 C CNN
+F 0 "#PWR7" H 4850 4450 30  0001 C CNN
 F 1 "VCC" H 4850 4450 30  0000 C CNN
 	1    4850 4350
